File: Main Board_Muon/ROCKSAT_Modules_V1.kicad_pcb (KiCad board)
At the start: 2 copper layers, 76.2 x 76.2 mm, 24 parts, among them J1 Pins 1-10, J2 Pins 11-20, U1 MC7805, U2 Opamp_Dual, U4 Arduino_MKR_Zero

Commit message: mounting holes fixed. Mosfet Tab Down. Module Ready.
Parts:
- removed REF** (x4): MountingHole_3.2mm_M3_DIN965_Pad, MountingHole:MountingHole_3.2mm_M3_DIN965_Pad
- added H1: MountingHole, MountingHole:MountingHole_3.2mm_M3, F.Cu at (129.7, 83.0)
- added H2: MountingHole, MountingHole:MountingHole_3.2mm_M3, F.Cu at (180.5, 82.7)
- added H3: MountingHole, MountingHole:MountingHole_3.2mm_M3, F.Cu at (172.1, 130.0)
- added H4: MountingHole, MountingHole:MountingHole_3.2mm_M3, F.Cu at (129.7, 122.4)
- U1: footprint Package_TO_SOT_THT:TO-220-3_Vertical -> Package_TO_SOT_THT:TO-220-3_Horizontal_TabDown

Commit message: Test Points Added
Parts:
- added TP1: TP5V, TestPoint:TestPoint_THTPad_D1.5mm_Drill0.7mm, B.Cu at (187.3, 88.1)
- added TP10: TPA_MUON, TestPoint:TestPoint_THTPad_D1.5mm_Drill0.7mm, B.Cu at (133.2, 94.7)
- added TP11: TPFB_Filter, TestPoint:TestPoint_THTPad_D1.5mm_Drill0.7mm, B.Cu at (162.7, 114.0)
- added TP12: TPU2A_Out, TestPoint:TestPoint_THTPad_D1.5mm_Drill0.7mm, B.Cu at (173.9, 120.3)
- added TP2: TP3.3V, TestPoint:TestPoint_THTPad_D1.5mm_Drill0.7mm, B.Cu at (190.4, 100.8)
- added TP3: TPRXin, TestPoint:TestPoint_THTPad_D1.5mm_Drill0.7mm, B.Cu at (189.3, 93.2)
- added TP4: TPTXin, TestPoint:TestPoint_THTPad_D1.5mm_Drill0.7mm, B.Cu at (163.2, 108.9)
- added TP5: TPMOSI, TestPoint:TestPoint_THTPad_D1.5mm_Drill0.7mm, B.Cu at (163.4, 125.4)
- added TP6: TPMISO, TestPoint:TestPoint_THTPad_D1.5mm_Drill0.7mm, B.Cu at (125.1, 92.1)
- added TP7: TPSCLK, TestPoint:TestPoint_THTPad_D1.5mm_Drill0.7mm, B.Cu at (132.7, 107.6)
- added TP8: TPGND, TestPoint:TestPoint_THTPad_D1.5mm_Drill0.7mm, B.Cu at (187.6, 105.6)
- added TP9: TPA_(+), TestPoint:TestPoint_THTPad_D1.5mm_Drill0.7mm, B.Cu at (172.8, 91.9)
Routing:
- net /MISO: track 39.7 -> 49.7 mm
- net /RX_IN: track 28.9 -> 37.7 mm
- net +3.3: track 66.5 -> 75.2 mm
- net /SCLK: track 39.7 -> 48.4 mm
- net +5V: track 111.7 -> 118.4 mm
- net /A_Muon: track 29.7 -> 35.9 mm
- net /MOSI: track 40.4 -> 46.4 mm
- net /TX_IN: track 29.4 -> 34.4 mm
- net /A_(+): track 20.8 -> 25.0 mm
- net /FB_Filter: track 16.7 -> 20.7 mm
- net /U2A_Out: track 19.9 -> 23.2 mm
