File: Main Board_Muon/ROCKSAT_Modules_V1.kicad_sch (KiCad schematic)
At the start: 20 parts, among them J1 Pins 1-10, J2 Pins 11-20, U1 MC7805, U2 Opamp_Dual, U4 Arduino_MKR_Zero

Commit message: mounting holes fixed. Mosfet Tab Down. Module Ready.
Parts:
- added H1, H2, H3, H4: MountingHole, MountingHole:MountingHole_3.2mm_M3, symbol Mechanical:MountingHole

Commit message: Test Points Added
Parts:
- added TP1: TP5V, TestPoint:TestPoint_THTPad_D1.5mm_Drill0.7mm, symbol Connector:TestPoint
- added TP10: TPA_MUON, TestPoint:TestPoint_THTPad_D1.5mm_Drill0.7mm, symbol Connector:TestPoint
- added TP11: TPFB_Filter, TestPoint:TestPoint_THTPad_D1.5mm_Drill0.7mm, symbol Connector:TestPoint
- added TP12: TPU2A_Out, TestPoint:TestPoint_THTPad_D1.5mm_Drill0.7mm, symbol Connector:TestPoint
- added TP2: TP3.3V, TestPoint:TestPoint_THTPad_D1.5mm_Drill0.7mm, symbol Connector:TestPoint
- added TP3: TPRXin, TestPoint:TestPoint_THTPad_D1.5mm_Drill0.7mm, symbol Connector:TestPoint
- added TP4: TPTXin, TestPoint:TestPoint_THTPad_D1.5mm_Drill0.7mm, symbol Connector:TestPoint
- added TP5: TPMOSI, TestPoint:TestPoint_THTPad_D1.5mm_Drill0.7mm, symbol Connector:TestPoint
- added TP6: TPMISO, TestPoint:TestPoint_THTPad_D1.5mm_Drill0.7mm, symbol Connector:TestPoint
- added TP7: TPSCLK, TestPoint:TestPoint_THTPad_D1.5mm_Drill0.7mm, symbol Connector:TestPoint
- added TP8: TPGND, TestPoint:TestPoint_THTPad_D1.5mm_Drill0.7mm, symbol Connector:TestPoint
- added TP9: TPA_(+), TestPoint:TestPoint_THTPad_D1.5mm_Drill0.7mm, symbol Connector:TestPoint
Connections:
- net +3.3: now also TP2.1
- net +5V: now also TP1.1
- net A_(+): now also TP9.1
- net A_Muon: now also TP10.1
- net FB_Filter: now also TP11.1
- net GND: now also TP8.1
- net MISO: now also TP6.1
- net MOSI: now also TP5.1
- net RX_IN: now also TP3.1
- net SCLK: now also TP7.1
- net TX_IN: now also TP4.1
- net U2A_Out: now also TP12.1

Commit message: BOM Updates
Parts:
- U4: now left out of the parts list
Changed lines of the file:
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@@
 			)
 		)
-		(property "Datasheet" "https://www.onsemi.cn/PowerSolutions/document/MC7800-D.PDF"
+		(property "Datasheet" "https://www.onsemi.com/pdf/datasheet/mc7800-d.pdf"
 			(at 118.11 83.82 0)
 			(effects
@@
 			)
 		)
-		(property "Description" "Positive 1A 35V Linear Regulator, Fixed Output 5V, TO-220"
+		(property "Description" "MC7805CTG"
 			(at 118.11 82.55 0)
 			(effects
@@
 		(unit 1)
 		(exclude_from_sim no)
-		(in_bom yes)
+		(in_bom no)
 		(on_board yes)
 		(dnp no)
@@
 			)
 		)
-		(property "Description" "Dual operational amplifier"
+		(property "Description" "LT1807CS8#PBF"
 			(at 217.17 71.12 0)
 			(effects
@@
 			)
 		)
-		(property "Description" "Dual operational amplifier"
+		(property "Description" "LT1807CS8#PBF"
 			(at 201.93 43.18 0)
 			(effects
@@
 			)
 		)
-		(property "Description" "Resistor"
+		(property "Description" "Wire"
 			(at 255.27 85.09 0)
 			(effects
@@
 			)
 		)
-		(property "Description" "Dual operational amplifier"
+		(property "Description" "LT1807CS8#PBF"
 			(at 181.61 68.58 0)
 			(effects

Commit message: BOM Completed 3-22-26
Parts:
- C3: Notes (none) -> 22nf
- C4: Notes (none) -> Wire; now left out of the parts list
- D1, D2: Notes (none) -> Not the same diode. should be similar
- J1, J2, R13: now left out of the parts list
- R10: Notes (none) -> Actual value 250
- R12: Notes (none) -> Actual value is 20k. dont think it will make a difference. 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
